Commit message: hiddening the link_b2 into urdf files Gazebo

File: invite_motoman_gazebo/urdf/urdf_src/motoman_csda10f_support/common_torso_macro.xacro (robot description, xacro)
@@ -118,4 +118,10 @@
 		</transmission>
 		<!-- end of transmission list -->
+        <!-- Gazebo-specific link properties -->
+		<gazebo reference="${prefix}link_b2">
+			<visual>
+				<transparency>1</transparency>
+			</visual>
+		</gazebo>
 	</xacro:macro>
 </robot>
