Commit message: v1.1.2 Robot interface enhancements, and reconfiguration of grippers
- Small changes in vision pipeline, message filtering is not being used any more to concatenate both cameras pointclouds.
- Addition of moveit visual tools instance on robot interface. 
- Moveit configuration changes.
- Delete old tutorials, start migration to robot interface usage.

File: invite_motoman_support/urdf/left_gripper_macro.xacro (robot description, xacro)
@@ -69,5 +69,6 @@
 				<origin rpy="0 0 0" xyz="0 0 0.0095"/>
 				<geometry>
-					<cylinder length="0.019" radius="0.043"/>
+					<!-- <cylinder length="0.019" radius="0.043"/> -->
+          <cylinder length="${0.05}" radius="${0.043 + 0.04}"/>
 				</geometry>
 				<material name="yellow"/>

File: invite_motoman_support/urdf/right_gripper_macro.xacro (robot description, xacro)
@@ -41,5 +41,5 @@
 				<origin rpy="${pi/2} 0 0" xyz="0 0.0045 0"/>
 				<geometry>
-					<cylinder length="0.009" radius="0.038"/>
+					<cylinder length="${0.009 + 0.03}" radius="${0.038 + 0.04}"/>
 				</geometry>
 				<material name="yellow"/>
