Commit message: v0.1.2 - Reconfigure grippers TCP`s, Change Rviz default configurations, modify move_group_interface_tutorial, and fix URDF

File: invite_motoman_support/urdf/invite_csda10f.xacro (robot description, xacro)
@@ -32,3 +32,15 @@
 		<axis xyz="0 0 1"/>
   	</joint>
+    <link name="arm_right_link_tcp" />
+	<link name="arm_left_link_tcp" />
+    <joint name="arm_right_joint_tcp" type="fixed" >
+      <origin xyz="0 0 0.1994" rpy="0 0 0"/>
+      <parent link="arm_right_link_tool0" />
+      <child link="arm_right_link_tcp" />
+    </joint>
+	<joint name="arm_left_joint_tcp" type="fixed" >
+      <origin xyz="0 0 0.2094" rpy="0 0 ${111.42*pi/180}"/>
+      <parent link="arm_left_link_tool0" />
+      <child link="arm_left_link_tcp" />
+    </joint>
 </robot>

Commit message: General corrections
* Create two new move groups `arm_left_torso` and `arm_right_torso`.
* Update left gripper position
* Create motion test Node file

File: invite_motoman_support/urdf/invite_csda10f.xacro (robot description, xacro)
@@ -24,5 +24,5 @@
     	<parent link="arm_left_link_tool0" />
     	<child link="arm_left_link_force_sensor_adapter_plate" />
-		<origin xyz="0 0 0" rpy="0 0 ${111.42*pi/180}"/>
+		<origin xyz="0 0 0" rpy="0 0 ${90*pi/180}"/>
 		<axis xyz="0 0 1"/>
  	 </joint>
@@ -43,5 +43,5 @@
     </joint>
 	<joint name="arm_left_joint_tcp" type="fixed" >
-      <origin xyz="0 0 0.2094" rpy="0 0 ${111.42*pi/180}"/>
+      <origin xyz="0 0 0.2094" rpy="0 0 ${90*pi/180}"/>
       <parent link="arm_left_link_tool0" />
       <child link="arm_left_link_tcp" />

Commit message: Correction on move_group configuration

File: invite_motoman_support/urdf/invite_csda10f.xacro (robot description, xacro)
@@ -47,3 +47,17 @@
       <child link="arm_left_link_tcp" />
     </joint>
+    <!--<link name="ensenso_upper_optical_frame" />
+    <link name="ensenso_lower_optical_frame" />
+	<joint name="upper_camera_joint" type="fixed" >
+      <origin xyz="0.77251 0.237802 1.89592" rpy="-2.89024 0.00537681 1.55567"/>
+      <parent link="base_link" />
+      <child link="ensenso_upper_optical_frame" />
+    </joint>
+	<joint name="lower_camera_joint" type="fixed" >
+      <origin xyz="0.613277 1.31721 1.44293" rpy="-1.98763 0.0018727 3.12335"/>
+      <parent link="base_link" />
+      <child link="ensenso_lower_optical_frame" />
+    </joint>-->
+	<!-- Q upper cammera   0.087429787325731 -0.7070500191913 -0.695960729680754 0.0898608112137424 -->
+	<!-- Q lower cammera   0.00419018865331527 -0.00815435540059931 -0.83807389015755 0.545479700303542 -->
 </robot>

Commit message: Vision V0.0.1 Initial configuration
- Ensenso N35 upper and lower cameras included in robot description
- Cameras Node and camera data request configured for both cameras.
- Moveit sensor configuration.

File: invite_motoman_support/urdf/invite_csda10f.xacro (robot description, xacro)
@@ -47,16 +47,16 @@
       <child link="arm_left_link_tcp" />
     </joint>
-    <!--<link name="ensenso_upper_optical_frame" />
+    <link name="ensenso_upper_optical_frame" />
     <link name="ensenso_lower_optical_frame" />
 	<joint name="upper_camera_joint" type="fixed" >
-      <origin xyz="0.77251 0.237802 1.89592" rpy="-2.89024 0.00537681 1.55567"/>
+      <origin xyz="0.875275 0.259338 1.89787" rpy="-2.89701 0.0272259 1.57315"/>
       <parent link="base_link" />
       <child link="ensenso_upper_optical_frame" />
     </joint>
 	<joint name="lower_camera_joint" type="fixed" >
-      <origin xyz="0.613277 1.31721 1.44293" rpy="-1.98763 0.0018727 3.12335"/>
+      <origin xyz="0.695186 1.32848 1.41829" rpy="-1.9854 -0.00862869 -3.13558"/>
       <parent link="base_link" />
       <child link="ensenso_lower_optical_frame" />
-    </joint>-->
+    </joint>
 	<!-- Q upper cammera   0.087429787325731 -0.7070500191913 -0.695960729680754 0.0898608112137424 -->
 	<!-- Q lower cammera   0.00419018865331527 -0.00815435540059931 -0.83807389015755 0.545479700303542 -->

Commit message: Update grippers and Robot URDF files
- Update of collision matrix
- Creation of left gripper URDF file
- Right gripper finger tips addition 
- Migration of Robotiq gripper package to this repository until the pull request is accepted by the `ros-industrial/robotiq` repository.

File: invite_motoman_support/urdf/invite_csda10f.xacro (robot description, xacro)
@@ -17,17 +17,17 @@
 	<xacro:motoman_csda10f prefix=""/>
 	<!--Create an instance of the right arm gripper macro-->
-  	<xacro:invite_csda10f_right_gripper prefix="arm_right_"/>
+  	<xacro:invite_csda10f_right_gripper prefix="right_gripper_"/>
 	<!--Create an instance of the right left gripper macro-->
-  	<xacro:invite_csda10f_left_gripper prefix="arm_left_"/>
+  	<xacro:invite_csda10f_left_gripper prefix="left_gripper_"/>
 <!--Joints joining the grippers to the robot-->
 	<joint name="left_gripper_to_robot_joint" type="fixed">
     	<parent link="arm_left_link_tool0" />
-    	<child link="arm_left_link_force_sensor_adapter_plate" />
+    	<child link="left_gripper_link_force_sensor_adapter_plate" />
 		<origin xyz="0 0 0" rpy="0 0 ${111.42*pi/180}"/>
 		<axis xyz="0 0 1"/>
  	 </joint>
-	<joint name="right_gripper_to_robot_joint" type="fixed">
+	<joint name="right_gripper__to_robot_joint" type="fixed">
 		<parent link="arm_right_link_tool0" />
-		<child link="arm_right_link_gripper_adapter_plate" />
+		<child link="right_gripper_link_gripper_adapter_plate" />
 		<origin xyz="0 0 0" rpy="${pi/2} 0 0"/>
 		<axis xyz="0 0 1"/>

File: invite_motoman_support/urdf/left_gripper_macro.xacro (robot description, xacro)
@@ -15,5 +15,5 @@
 	<xacro:macro name="invite_csda10f_left_gripper" params="prefix">
 		<!--Import macro from 2-finger adaptative robotiq gripper-->
-		<xacro:include filename="$(find robotiq_2f_model)/model/robotiq_2f_85.urdf.xacro" />
+		<xacro:include filename="$(find robotiq_2f_85_gripper_visualization)/urdf/robotiq_arg2f_85_model_macro.xacro" />
 <!--LINKS********************************************************************************************************************************-->
 		<!--Aluminium Adapter plate for Robotiq coupling and CSDA10F arm flange-->
@@ -93,5 +93,7 @@
 			</collision>
 		</link>-->
-<!--Joints ******************************************************************************************************************-->
+		<!-- Instance of C3 85mm Model  -->
+		<xacro:robotiq_arg2f_85 prefix="${prefix}"/>
+	<!--Joints ******************************************************************************************************************-->
 		<!--Joint force sensor adaptor plate to force sensor-->
 		<joint name="${prefix}gripper_flange_joint" type="fixed">
@@ -112,8 +114,10 @@
 			<child link="${prefix}link_robotiq_coupling" />
 		</joint>
-		<!--ROBOTIQ 85mm Gripper instance creation-->
-		<xacro:robotiq_2f_85 name="arm_left" parent="${prefix}link_robotiq_coupling" precise_collision="false" adaptive_transmission="false">
+		<!--Joint from the robotiq coupling to the gripper itself-->
+		<joint name="${prefix}joint" type="fixed">
 			<origin xyz="0 0 0.0039" rpy="0 0 ${pi}"/>
-		</xacro:robotiq_2f_85>
+			<parent link="${prefix}link_robotiq_coupling" />
+			<child link="${prefix}robotiq_arg2f_base_link" />
+		</joint>
 	</xacro:macro>
 </robot>

File: invite_motoman_support/urdf/right_gripper_macro.xacro (robot description, xacro)
@@ -26,5 +26,5 @@
 	<xacro:macro name="invite_csda10f_right_gripper" params="prefix">
 		<!--Import macro from 2-finger adaptative robotiq gripper-->
-		<xacro:include filename="$(find robotiq_arg2f_model_visualization)/urdf/robotiq_arg2f_140_model_macro.xacro" />
+		<xacro:include filename="$(find robotiq_2f_140_gripper_visualization)/urdf/robotiq_arg2f_140_model_macro.xacro" />
 		<!--Aluminium Adapter plate for Robotiq coupling and CSDA10F arm flange-->
 		<link name="${prefix}link_gripper_adapter_plate">
@@ -65,7 +65,9 @@
 			</collision>
 		</link>-->
-		<xacro:robotiq_arg2f_140 prefix="right_gripper_"/>
+		<!-- Instance of C3 140mm Model  -->
+		<xacro:robotiq_arg2f_140 prefix="${prefix}"/>
+	<!--Joints ******************************************************************************************************************-->
 		<!--Joint from the adapter plate to the robotiq gripper coupling-->
-		<joint name="right_gripper_gripper_coupling_joint" type="fixed">
+		<joint name="${prefix}gripper_coupling_joint" type="fixed">
 			<origin  xyz="0 0.0160 0" rpy="${-pi/2} 0 0"/>
 			<parent link="${prefix}link_gripper_adapter_plate" />
@@ -73,8 +75,8 @@
 		</joint>
 		<!--Joint from the robotiq coupling to the gripper itself-->
-		<joint name="right_gripper_joint" type="fixed">
+		<joint name="${prefix}joint" type="fixed">
 			<origin xyz="0 0.0 0.0039" rpy="0 0 ${pi}" />
 			<parent link="${prefix}link_robotiq_coupling" />
-			<child link="right_gripper_robotiq_arg2f_base_link" />
+			<child link="${prefix}robotiq_arg2f_base_link" />
 		</joint>
 	</xacro:macro>

Commit message: v1.0.3 Modification of control interface for Robotiq grippers
Based on the package from [waypointrobotics/robotiq_85_gripper](https://github.com/waypointrobotics/robotiq_85_gripper), a control interface of both Robotiq grippers (140mm and 85mm) was developed, allowing to control the grippers through the use of an Action Client.
Whats new: 
- Action Client-Server structure developed for control of multiple robotiq grippers.
- Publication of real-time gripper joint state.

This packages should migrate in the future to an independent repository or to the robotiq ros-industrial repository.

File: invite_motoman_support/urdf/invite_csda10f.xacro (robot description, xacro)
@@ -30,5 +30,5 @@
 		<parent link="arm_right_link_tool0" />
 		<child link="right_gripper_link_gripper_adapter_plate" />
-		<origin xyz="0 0 0" rpy="${pi/2} 0 0"/>
+		<origin xyz="0 0 0" rpy="${pi/2} 0 ${pi/2}"/>
 		<axis xyz="0 0 1"/>
   	</joint>

File: robotiq_2finger_grippers/robotiq_2f_140_gripper_visualization/urdf/robotiq_arg2f_140_model_macro.xacro (robot description, xacro)
@@ -188,5 +188,5 @@
       <child link="${prefix}left_outer_knuckle" />
       <axis xyz="-1 0 0" />
-      <limit lower="0" upper="0.775" velocity="2.0" effort="1000" />
+      <limit lower="0" upper="0.7" velocity="2.0" effort="1000" />
     </joint>
     <xacro:finger_joints prefix="${prefix}" fingerprefix="left" reflect="1.0"/>

File: robotiq_2finger_grippers/robotiq_2f_85_gripper_visualization/urdf/robotiq_arg2f_85_model.xacro (robot description, xacro)
@@ -2,4 +2,4 @@
 <robot name="robotiq_arg2f_85_model" xmlns:xacro="http://ros.org/wiki/xacro">
   <xacro:include filename="$(find robotiq_2f_85_gripper_visualization)/urdf/robotiq_arg2f_85_model_macro.xacro" />
-  <xacro:robotiq_arg2f_85 prefix=""/>
+  <xacro:robotiq_arg2f_85 prefix="prefix"/>
 </robot>

Commit message: v1.0.4 Addition of Robotiq Control scripts and configuration
Plus general bug fixing

File: invite_motoman_support/urdf/invite_csda10f.xacro (robot description, xacro)
@@ -50,10 +50,12 @@
     <link name="ensenso_lower_optical_frame" />
 	<joint name="upper_camera_joint" type="fixed" >
-      <origin xyz="0.77251 0.237802 1.89592" rpy="-2.89024 0.00537681 1.55567"/>
+      <origin xyz="0.865275 0.259338 1.89787" rpy="-2.89701 0.0272259 1.57315"/>
+      <!-- <origin xyz="0.875275 0.259338 1.89787" rpy="-2.89701 0.0272259 1.57315"/> -->
       <parent link="base_link" />
       <child link="ensenso_upper_optical_frame" />
     </joint>
 	<joint name="lower_camera_joint" type="fixed" >
-      <origin xyz="0.613277 1.31721 1.44293" rpy="-1.98763 0.0018727 3.12335"/>
+      <origin xyz="0.685186 1.32848 1.41829" rpy="-1.9854 -0.00862869 -3.13558"/>
+      <!-- <origin xyz="0.695186 1.32848 1.41829" rpy="-1.9854 -0.00862869 -3.13558"/> -->
       <parent link="base_link" />
       <child link="ensenso_lower_optical_frame" />

Commit message: v1.1.0 New `CSDA10F` and `VisionInterface` classes
- new `csda10f_interface.h`: Defines the CSDA10F class which permits fast initialization, configuration and control of Robot motion groups and grippers. 
- new `vision_system_interface.h`: File defines the class `VisionInterface` which allows for easy initialization and control over the robot IDS N35 cameras. 
- Two new move groups (each arm + torso) to have a 8 DoF arm group.
- Default `RRTConnect` parameters setup

File: invite_motoman_support/urdf/invite_csda10f.xacro (robot description, xacro)
@@ -34,14 +34,14 @@
   	</joint>
 <!--Define the TCP of the grippers -->
-    <link name="arm_right_link_tcp" />
+  <link name="arm_right_link_tcp" />
 	<link name="arm_left_link_tcp" />
 <!--Define the position of the TCP with respect to the arm flange-->
     <joint name="arm_right_joint_tcp" type="fixed" >
-      <origin xyz="0 0 0.1994" rpy="0 0 0"/>
+      <origin xyz="0 0 ${0.1994 + 0.03}" rpy="0 0 ${pi/2}"/>
       <parent link="arm_right_link_tool0" />
       <child link="arm_right_link_tcp" />
     </joint>
 	<joint name="arm_left_joint_tcp" type="fixed" >
-      <origin xyz="0 0 0.2094" rpy="0 0 ${111.42*pi/180}"/>
+      <origin xyz="0 0 ${0.2094 + 0.03}" rpy="0 0 ${111.42*pi/180}"/>
       <parent link="arm_left_link_tool0" />
       <child link="arm_left_link_tcp" />

Commit message: v1.1.1 Logging level and minor configuration changes

File: invite_motoman_support/urdf/invite_csda10f.xacro (robot description, xacro)
@@ -43,5 +43,5 @@
     </joint>
 	<joint name="arm_left_joint_tcp" type="fixed" >
-      <origin xyz="0 0 ${0.2094 + 0.03}" rpy="0 0 ${111.42*pi/180}"/>
+      <origin xyz="0 0 ${0.2094 + 0.01}" rpy="0 0 ${111.42*pi/180}"/>
       <parent link="arm_left_link_tool0" />
       <child link="arm_left_link_tcp" />

Commit message: v1.1.4 Update in documentation - Change of gripper setup

File: invite_motoman_support/urdf/invite_csda10f.xacro (robot description, xacro)
@@ -23,6 +23,6 @@
 	<joint name="left_gripper_to_robot_joint" type="fixed">
     	<parent link="arm_left_link_tool0" />
-    	<child link="left_gripper_link_force_sensor_adapter_plate" />
-		<origin xyz="0 0 0" rpy="0 0 ${111.42*pi/180}"/>
+    	<child link="left_gripper_link_gripper_adapter_plate" />
+		<origin xyz="0 0 0" rpy="0 0 0"/>
 		<axis xyz="0 0 1"/>
  	 </joint>
@@ -38,17 +38,50 @@
 <!--Define the position of the TCP with respect to the arm flange-->
     <joint name="arm_right_joint_tcp" type="fixed" >
-      <origin xyz="0 0 ${0.1994 + 0.03}" rpy="0 0 ${pi/2}"/>
+      <origin xyz="0 0 ${0.1994 - 0.059 + 0.015}" rpy="0 0 ${pi/2}"/>
       <parent link="arm_right_link_tool0" />
       <child link="arm_right_link_tcp" />
     </joint>
 	<joint name="arm_left_joint_tcp" type="fixed" >
-      <origin xyz="0 0 ${0.2094 + 0.01}" rpy="0 0 ${111.42*pi/180}"/>
+      <origin xyz="0 0 ${0.2094 + 0.01 - 0.059}" rpy="0 0 0"/>
       <parent link="arm_left_link_tool0" />
       <child link="arm_left_link_tcp" />
     </joint>
-    <link name="ensenso_upper_optical_frame" />
-    <link name="ensenso_lower_optical_frame" />
+	<link name="ensenso_upper_optical_frame">
+		<visual>
+			<origin rpy="0 0 0" xyz="0 0 0"/>
+			<geometry>
+				<box size="0.4 0.25 0.25"/>
+			</geometry>
+			<material name="ensenso_color">
+						<color rgba="0.0 0.2 0.7 0.7"/>
+			</material>
+		</visual>
+		<collision>
+			<origin rpy="0 0 0" xyz="0 0 0"/>
+			<geometry>
+				<box size="0.4 0.25 0.25"/>
+			</geometry>
+		</collision>
+	</link>
+	<link name="ensenso_lower_optical_frame">
+		<visual>
+			<origin rpy="0 0 0" xyz="0 0 0"/>
+			<geometry>
+				<box size="0.4 0.25 0.25"/>
+			</geometry>
+			<material name="ensenso_color">
+						<color rgba="0.0 0.2 0.7 0.7"/>
+			</material>
+		</visual>
+		<collision>
+			<origin rpy="0 0 0" xyz="0 0 0"/>
+			<geometry>
+				<box size="0.4 0.25 0.25"/>
+			</geometry>
+		</collision>
+	</link>
 	<joint name="upper_camera_joint" type="fixed" >
-      <origin xyz="0.865275 0.259338 1.89787" rpy="-2.89701 0.0272259 1.57315"/>
+      <origin xyz="0.860775 0.265338 1.88787" rpy="-2.89701 0.0272259 1.57315"/>
+      <!-- <origin xyz="0.865275 0.259338 1.89787" rpy="-2.89701 0.0272259 1.57315"/> -->
       <!-- <origin xyz="0.875275 0.259338 1.89787" rpy="-2.89701 0.0272259 1.57315"/> -->
       <parent link="base_link" />
@@ -62,4 +95,27 @@
     </joint>
 	<!-- Q upper cammera   0.087429787325731 -0.7070500191913 -0.695960729680754 0.0898608112137424 -->
-	<!-- Q lower cammera   0.00419018865331527 -0.00815435540059931 -0.83807389015755 0.545479700303542 -->
+	<!-- Q lower cammera   0.00419018865331527 -0.00815435540059931 -0.83807389015755
+	0.545479700303542 -->
+	<!-- Define lifting rings collision objects -->
+	<link name="lifting_rings">
+		<visual>
+			<origin rpy="0 0 0" xyz="0 0 0"/>
+			<geometry>
+				<box size="0.0001 0.0001 0.0001"/>
+			</geometry>
+			<!-- <material name="yellow"/> -->
+		</visual>
+		<collision>
+			<origin rpy="0 0 0" xyz="0 0 0"/>
+			<geometry>
+				<box size="0.055 0.17 0.075"/>
+			</geometry>
+			<material name="yellow"/>
+		</collision>
+	</link>
+	<joint name="lifting_rings_joint" type="fixed">
+		<origin xyz="0.1 0.0 0.515" rpy="0 0 0"/>
+		<parent link="torso_link_b1" />
+		<child link="lifting_rings" />
+	</joint>
 </robot>

File: invite_motoman_support/urdf/left_gripper.xacro (robot description, xacro)
@@ -11,5 +11,5 @@
   <xacro:include filename="$(find invite_motoman_support)/urdf/left_gripper_macro.xacro" />
   <!--Create an instance of the left arm gripper macro-->
-  <xacro:invite_csda10f_left_gripper prefix="arm_left_"/>
+  <xacro:invite_csda10f_left_gripper prefix=""/>
   <!--Base frame for reference-->
   <link name="base_link" />
@@ -17,5 +17,5 @@
   <joint name="world_joint" type="fixed">
     <parent link="base_link" />
-    <child link="arm_left_link_force_sensor_adapter_plate" />
+    <child link="link_gripper_adapter_plate" />
     <origin xyz="0 0 0" rpy="0 0 0"/>
     <axis xyz="0 0 1"/>

File: invite_motoman_support/urdf/left_gripper_macro.xacro (robot description, xacro)
@@ -20,5 +20,5 @@
 		<link name="${prefix}link_gripper_adapter_plate">
 			<visual>
-				<origin rpy="0 0 0" xyz="0 0 0"/>
+				<origin rpy="${pi/2} 0 0" xyz="0 0 0"/>
 				<geometry>
 					<mesh filename="package://invite_motoman_support/meshes/robotiq-yaskawa_adapter_plate.stl" scale="0.001 0.001 0.001"/>
@@ -55,61 +55,10 @@
 			</collision>
 		</link>-->
-		<!--Dynpick adaptor plate, which connects the force sensor with the robot flange-->
-		<link name="${prefix}link_force_sensor_adapter_plate">
-			<visual>
-				<origin rpy="0 0 0" xyz="0.00 0 0.0095"/>
-				<geometry>
-					<cylinder length="0.019" radius="0.043"/>
-				</geometry>
-				<material name="aluminium">
-  			        <color rgba="0.917 0.917 0.917 1.0"/>
-  				</material>
-			</visual>
-			<collision>
-				<origin rpy="0 0 0" xyz="0 0 0.0095"/>
-				<geometry>
-					<!-- <cylinder length="0.019" radius="0.043"/> -->
-          <cylinder length="${0.05}" radius="${0.043 + 0.04}"/>
-				</geometry>
-				<material name="yellow"/>
-			</collision>
-		</link>-->
-		<!--Dynpick adaptor plate, which connects the force sensor with the robot flange-->
-		<link name="${prefix}link_force_sensor">
-			<visual>
-				<origin rpy="0 0 0" xyz="0 0 0"/>
-				<geometry>
-					<cylinder length="0.040" radius="0.045"/>
-				</geometry>
-				<material name="red-aluminium">
-  			        <color rgba="0.721 0 0 1.0"/>
-  				</material>
-			</visual>
-			<collision>
-				<origin rpy="0 0 0" xyz="0 0 0"/>
-				<geometry>
-					<cylinder length="0.040" radius="0.0455"/>
-				</geometry>
-				<material name="yellow"/>
-			</collision>
-		</link>-->
 		<!-- Instance of C3 85mm Model  -->
 		<xacro:robotiq_arg2f_85 prefix="${prefix}"/>
 	<!--Joints ******************************************************************************************************************-->
-		<!--Joint force sensor adaptor plate to force sensor-->
-		<joint name="${prefix}gripper_flange_joint" type="fixed">
-			<origin  xyz="0 0 0.039" rpy="0 0 0"/>
-			<parent link="${prefix}link_force_sensor_adapter_plate" />
-			<child link="${prefix}link_force_sensor" />
-		</joint>
-		<!--Joint from the force sensor to the gripper adaptor plate-->
-		<joint name="${prefix}gripper_force_sensor_joint" type="fixed">
-			<origin  xyz="0 0 0.02" rpy="${pi/2} 0 0"/>
-			<parent link="${prefix}link_force_sensor" />
-			<child link="${prefix}link_gripper_adapter_plate" />
-		</joint>
 		<!--Joint from the adapter plate to the robotiq gripper coupling-->
 		<joint name="${prefix}gripper_coupling_joint" type="fixed">
-			<origin  xyz="0 0.0160 0" rpy="${-pi/2} 0 0"/>
+			<origin  xyz="0 0 0.0160" rpy="0 0 0"/>
 			<parent link="${prefix}link_gripper_adapter_plate" />
 			<child link="${prefix}link_robotiq_coupling" />

File: invite_motoman_support/urdf/right_gripper_macro.xacro (robot description, xacro)
@@ -26,5 +26,5 @@
 	<xacro:macro name="invite_csda10f_right_gripper" params="prefix">
 		<!--Import macro from 2-finger adaptative robotiq gripper-->
-		<xacro:include filename="$(find robotiq_2f_140_gripper_visualization)/urdf/robotiq_arg2f_140_model_macro.xacro" />
+		<xacro:include filename="$(find robotiq_2f_85_gripper_visualization)/urdf/robotiq_arg2f_85_model_macro.xacro" />
 		<!--Aluminium Adapter plate for Robotiq coupling and CSDA10F arm flange-->
 		<link name="${prefix}link_gripper_adapter_plate">
@@ -66,5 +66,5 @@
 		</link>-->
 		<!-- Instance of C3 140mm Model  -->
-		<xacro:robotiq_arg2f_140 prefix="${prefix}"/>
+		<xacro:robotiq_arg2f_85 prefix="${prefix}"/>
 	<!--Joints ******************************************************************************************************************-->
 		<!--Joint from the adapter plate to the robotiq gripper coupling-->
