Commit message: v1.1.5 Config of FT300 sensor, general config updates
Addition of URDF models to fix the FT300 sensor to the robot arm.
Add functionalities to stop the robot motion on and to tare the new force/torque sensor on command in the `CSDA10F Interface` class

- Removal of trash code and files

File: invite_motoman_support/urdf/invite_csda10f.xacro (robot description, xacro)
@@ -5,46 +5,46 @@
 		both 2-Finger Adaptative Robotiq Grippers (140mm one for the right arm and 80mm one for the left one)
 -->
-<robot name="motoman_csda10f" xmlns:xacro="http://ros.org/wiki/xacro">
-<!-- Import macros required-->
+<robot name="motoman_csda10f"
+	xmlns:xacro="http://ros.org/wiki/xacro">
+	<!-- Import macros required-->
 	<!--Import macro for the CSDA10F robot-->
 	<xacro:include filename="$(find motoman_csda10f_support)/urdf/csda10f_macro.xacro" />
 	<!--Import macro for left arm gripper-->
-  	<xacro:include filename="$(find invite_motoman_support)/urdf/left_gripper_macro.xacro" />
-  	<!--Import macro for right arm gripper-->
-  	<xacro:include filename="$(find invite_motoman_support)/urdf/right_gripper_macro.xacro" />
-<!--Create instance of the macros imported-->
+	<xacro:include filename="$(find invite_motoman_support)/urdf/left_gripper_macro.xacro" />
+	<!--Import macro for right arm gripper-->
+	<xacro:include filename="$(find invite_motoman_support)/urdf/right_gripper_macro.xacro" />
+	<!--Create instance of the macros imported-->
 	<!--Create an instance of YASKAWA Motoman CSDA10F robot-->
 	<xacro:motoman_csda10f prefix=""/>
 	<!--Create an instance of the right arm gripper macro-->
-  	<xacro:invite_csda10f_right_gripper prefix="right_gripper_"/>
+	<xacro:invite_csda10f_right_gripper prefix="right_gripper_"/>
 	<!--Create an instance of the right left gripper macro-->
-  	<xacro:invite_csda10f_left_gripper prefix="left_gripper_"/>
-<!--Joints joining the grippers to the robot-->
+	<xacro:invite_csda10f_left_gripper prefix="left_gripper_"/>
+	<!--Joints joining the grippers to the robot-->
 	<joint name="left_gripper_to_robot_joint" type="fixed">
-    	<parent link="arm_left_link_tool0" />
-    	<child link="left_gripper_link_gripper_adapter_plate" />
-		<origin xyz="0 0 0" rpy="0 0 0"/>
+		<parent link="arm_left_link_tool0" />
+		<child link="left_gripper_ft300_adapter_plate" />
+		<origin xyz="0 0 0" rpy="0 0 ${pi}"/>
 		<axis xyz="0 0 1"/>
- 	 </joint>
+	</joint>
 	<joint name="right_gripper__to_robot_joint" type="fixed">
 		<parent link="arm_right_link_tool0" />
-		<child link="right_gripper_link_gripper_adapter_plate" />
+		<child link="right_gripper_gripper_adapter_plate" />
 		<origin xyz="0 0 0" rpy="${pi/2} 0 ${pi/2}"/>
 		<axis xyz="0 0 1"/>
-  	</joint>
-<!--Define the TCP of the grippers -->
-  <link name="arm_right_link_tcp" />
+	</joint>
+	<!--Define the TCP of the grippers -->
+	<link name="arm_right_link_tcp" />
 	<link name="arm_left_link_tcp" />
-<!--Define the position of the TCP with respect to the arm flange-->
-    <joint name="arm_right_joint_tcp" type="fixed" >
-      <origin xyz="0 0 ${0.1994 - 0.059 + 0.015}" rpy="0 0 ${pi/2}"/>
-      <parent link="arm_right_link_tool0" />
-      <child link="arm_right_link_tcp" />
-    </joint>
-	<joint name="arm_left_joint_tcp" type="fixed" >
-      <origin xyz="0 0 ${0.2094 + 0.01 - 0.059}" rpy="0 0 0"/>
-      <parent link="arm_left_link_tool0" />
-      <child link="arm_left_link_tcp" />
-    </joint>
+	<joint name="arm_right_joint_tcp" type="fixed">
+		<origin xyz="0 0 ${0.1994 - 0.059 + 0.015}" rpy="0 0 ${pi/2}"/>
+		<parent link="arm_right_link_tool0" />
+		<child link="arm_right_link_tcp" />
+	</joint>
+	<joint name="arm_left_joint_tcp" type="fixed">
+		<origin xyz="0 0 ${0.21}" rpy="0 0 ${(50 + 90)*pi/180}"/>
+		<parent link="arm_left_link_tool0" />
+		<child link="arm_left_link_tcp" />
+	</joint>
 	<link name="ensenso_upper_optical_frame">
 		<visual>
@@ -54,5 +54,5 @@
 			</geometry>
 			<material name="ensenso_color">
-						<color rgba="0.0 0.2 0.7 0.7"/>
+				<color rgba="0.0 0.2 0.7 0.7"/>
 			</material>
 		</visual>
@@ -71,5 +71,5 @@
 			</geometry>
 			<material name="ensenso_color">
-						<color rgba="0.0 0.2 0.7 0.7"/>
+				<color rgba="0.0 0.2 0.7 0.7"/>
 			</material>
 		</visual>
@@ -81,41 +81,19 @@
 		</collision>
 	</link>
-	<joint name="upper_camera_joint" type="fixed" >
-      <origin xyz="0.860775 0.265338 1.88787" rpy="-2.89701 0.0272259 1.57315"/>
-      <!-- <origin xyz="0.865275 0.259338 1.89787" rpy="-2.89701 0.0272259 1.57315"/> -->
-      <!-- <origin xyz="0.875275 0.259338 1.89787" rpy="-2.89701 0.0272259 1.57315"/> -->
-      <parent link="base_link" />
-      <child link="ensenso_upper_optical_frame" />
-    </joint>
-	<joint name="lower_camera_joint" type="fixed" >
-      <origin xyz="0.685186 1.32848 1.41829" rpy="-1.9854 -0.00862869 -3.13558"/>
-      <!-- <origin xyz="0.695186 1.32848 1.41829" rpy="-1.9854 -0.00862869 -3.13558"/> -->
-      <parent link="base_link" />
-      <child link="ensenso_lower_optical_frame" />
-    </joint>
+	<joint name="upper_camera_joint" type="fixed">
+		<origin xyz="0.860775 0.265338 1.88787" rpy="-2.89701 0.0272259 1.57315"/>
+		<!-- <origin xyz="0.865275 0.259338 1.89787" rpy="-2.89701 0.0272259 1.57315"/> -->
+		<!-- <origin xyz="0.875275 0.259338 1.89787" rpy="-2.89701 0.0272259 1.57315"/> -->
+		<parent link="base_link" />
+		<child link="ensenso_upper_optical_frame" />
+	</joint>
+	<joint name="lower_camera_joint" type="fixed">
+		<origin xyz="0.685186 1.32848 1.41829" rpy="-1.9854 -0.00862869 -3.13558"/>
+		<!-- <origin xyz="0.695186 1.32848 1.41829" rpy="-1.9854 -0.00862869 -3.13558"/> -->
+		<parent link="base_link" />
+		<child link="ensenso_lower_optical_frame" />
+	</joint>
 	<!-- Q upper cammera   0.087429787325731 -0.7070500191913 -0.695960729680754 0.0898608112137424 -->
 	<!-- Q lower cammera   0.00419018865331527 -0.00815435540059931 -0.83807389015755
 	0.545479700303542 -->
-	<!-- Define lifting rings collision objects -->
-	<link name="lifting_rings">
-		<visual>
-			<origin rpy="0 0 0" xyz="0 0 0"/>
-			<geometry>
-				<box size="0.0001 0.0001 0.0001"/>
-			</geometry>
-			<!-- <material name="yellow"/> -->
-		</visual>
-		<collision>
-			<origin rpy="0 0 0" xyz="0 0 0"/>
-			<geometry>
-				<box size="0.055 0.17 0.075"/>
-			</geometry>
-			<material name="yellow"/>
-		</collision>
-	</link>
-	<joint name="lifting_rings_joint" type="fixed">
-		<origin xyz="0.1 0.0 0.515" rpy="0 0 0"/>
-		<parent link="torso_link_b1" />
-		<child link="lifting_rings" />
-	</joint>
 </robot>

File: invite_motoman_support/urdf/left_gripper_macro.xacro (robot description, xacro)
@@ -8,6 +8,4 @@
 	for example the adapter plate or the gripper itself).
 INTRUCTIONS:
-	The "Gripper base link" that is used to connect to the robot is:
-		'[your_gripper_prefix]link_force_sensor_adapter_plate'
 	An example on how to use this macro is shown in the file: 'left_gripper.xacro', of this same package
 -->
@@ -16,34 +14,72 @@
 		<!--Import macro from 2-finger adaptative robotiq gripper-->
 		<xacro:include filename="$(find robotiq_2f_85_gripper_visualization)/urdf/robotiq_arg2f_85_model_macro.xacro" />
-<!--LINKS********************************************************************************************************************************-->
-		<!--Aluminium Adapter plate for Robotiq coupling and CSDA10F arm flange-->
-		<link name="${prefix}link_gripper_adapter_plate">
+		<!-- Import macro of Robotiq force sensor FT300 -->
+		<xacro:include filename="$(find robotiq_ft_sensor)/urdf/robotiq_ft300.urdf.xacro" />
+		<!--LINKS********************************************************************************************************************************-->
+		<!--Aluminium Adapter plate from Flange to Robotiq Force Sensor adapter plate-->
+		<link name="${prefix}ft300_adapter_plate">
 			<visual>
-				<origin rpy="${pi/2} 0 0" xyz="0 0 0"/>
+				<origin xyz="0 0 0" rpy="0 ${-pi/2} ${pi/2}"/>
 				<geometry>
-					<mesh filename="package://invite_motoman_support/meshes/robotiq-yaskawa_adapter_plate.stl" scale="0.001 0.001 0.001"/>
+					<mesh filename="package://invite_motoman_support/meshes/visual/Adaptor-Flange-FT300.stl"/>
 				</geometry>
 				<material name="Aluminium">
-  			        <color rgba="0.816 0.816 0.816 1.0"/>
-  				</material>
+					<color rgba="0.816 0.816 0.816 1.0"/>
+				</material>
 			</visual>
 			<collision>
-				<origin rpy="${pi/2} 0 0" xyz="0 0.0045 0"/>
+				<!-- <origin xyz="0 0 0" rpy="0 ${-pi/2} ${pi/2}"/>
 				<geometry>
-					<cylinder length="0.009" radius="0.038"/>
+					<mesh filename="package://invite_motoman_support/meshes/collision/Adaptor-Flange-FT300.stl"/>
+				</geometry> -->
+				<geometry>
+					<cylinder length="${0.15}" radius="${0.038 + 0.04}"/>
 				</geometry>
-				<material name="yellow"/>
 			</collision>
+			<inertial>
+				<origin xyz="0 0 0.07" rpy="0 0 0"/>
+				<mass value="0.1356"/>
+				<inertia ixx="${(1/12)*0.1356*(0.014*0.014)}"
+								 iyy="${(1/12)*0.1356*(0.014*0.014)}"
+								 izz="${(1/2)*0.1356*(0.04*0.04 + 0.016*0.016)}"
+								 ixy="0" ixz="0" iyz="0"/>
+			</inertial>
 		</link>
-		<!--Robotiq coupling, that connects the gripper with the Adapter plate; this part host the cable connections of the gripper-->
-		<link name="${prefix}link_robotiq_coupling">
+		<!--Aluminium Adapter plate from Robotiq Force Sensor to Robotiq Gripper adapter plate-->
+		<link name="${prefix}gripper_adapter_plate">
 			<visual>
 				<origin rpy="0 0 0" xyz="0 0 0"/>
 				<geometry>
-					<mesh filename="package://invite_motoman_support/meshes/robotiq_gripper_coupling.stl" scale="0.001 0.001 0.001"/>
+					<mesh filename="package://invite_motoman_support/meshes/visual/Adaptor-FT300-Gripper.stl"/>
+				</geometry>
+				<material name="Aluminium">
+					<color rgba="0.816 0.816 0.816 1.0"/>
+				</material>
+			</visual>
+			<collision>
+				<origin rpy="0 0 0" xyz="0 0 0"/>
+				<geometry>
+					<mesh filename="package://invite_motoman_support/meshes/collision/Adaptor-FT300-Gripper.stl"/>
+				</geometry>
+			</collision>
+			<inertial>
+				<origin xyz="0 0 0.065" rpy="0 0 0"/>
+				<mass value="0.153"/>
+				<inertia ixx="${(1/12)*0.153*(0.012*0.012)}"
+								 iyy="${(1/12)*0.153*(0.012*0.012)}"
+								 izz="${(1/2)*0.153*(0.0375*0.0375)}"
+								 ixy="0" ixz="0" iyz="0" />
+			</inertial>
+		</link>
+		<!--Robotiq coupling, that connects the gripper with the Adapter plate; this part host the cable connections of the gripper-->
+		<link name="${prefix}robotiq_gripper_coupling">
+			<visual>
+				<origin rpy="0 0 0" xyz="0 0 0"/>
+				<geometry>
+					<mesh filename="package://invite_motoman_support/meshes/visual/robotiq_gripper_coupling.stl" scale="0.001 0.001 0.001"/>
 				</geometry>
 				<material name="light_balck">
-  			        <color rgba="0.17 0.17 0.17 1.0"/>
-  				</material>
+					<color rgba="0.17 0.17 0.17 1.0"/>
+				</material>
 			</visual>
 			<collision>
@@ -55,17 +91,28 @@
 			</collision>
 		</link>-->
-		<!-- Instance of C3 85mm Model  -->
+		<!-- Instance Gripper C3 85mm Model  -->
 		<xacro:robotiq_arg2f_85 prefix="${prefix}"/>
-	<!--Joints ******************************************************************************************************************-->
+		<!-- Instance FT300 Force Torque Sensor   -->
+		<xacro:robotiq_ft300 parent="${prefix}ft300_adapter_plate" prefix="${prefix}">
+			<origin xyz="0 0 0.010" rpy="0 0 ${25 * pi/180}"/>
+		</xacro:robotiq_ft300>
+		<!--Joints ******************************************************************************************************************-->
+		<!-- The joint from the ft300 coupling to the ft300 is defined in the
+		ft300 urdf -->
 		<!--Joint from the adapter plate to the robotiq gripper coupling-->
-		<joint name="${prefix}gripper_coupling_joint" type="fixed">
-			<origin  xyz="0 0 0.0160" rpy="0 0 0"/>
-			<parent link="${prefix}link_gripper_adapter_plate" />
-			<child link="${prefix}link_robotiq_coupling" />
+		<joint name="${prefix}gripper_adapter_plate_joint" type="fixed">
+			<origin xyz="0 0 0" rpy="0 0 ${(-90-20)*pi/180}"/>
+			<parent link="${prefix}robotiq_ft_frame_id" />
+			<child link="${prefix}gripper_adapter_plate" />
 		</joint>
-		<!--Joint from the robotiq coupling to the gripper itself-->
-		<joint name="${prefix}joint" type="fixed">
-			<origin xyz="0 0 0.0039" rpy="0 0 ${pi}"/>
-			<parent link="${prefix}link_robotiq_coupling" />
+		<!--Joint from the FT Sensor to the Gripper adaptor plate -->
+		<joint name="${prefix}robotiq_gripper_coupling_joint" type="fixed">
+			<origin xyz="0 0 ${0.012 + (0.0135/2)}" rpy="0 0 ${45*pi/180}"/>
+			<parent link="${prefix}gripper_adapter_plate" />
+			<child link="${prefix}robotiq_gripper_coupling" />
+		</joint>
+		<joint name="${prefix}robotiq_arg2f_joint" type="fixed">
+			<origin xyz="0 0 0.0039" rpy="0 0 ${pi/2}"/>
+			<parent link="${prefix}robotiq_gripper_coupling" />
 			<child link="${prefix}robotiq_arg2f_base_link" />
 		</joint>

File: invite_motoman_support/urdf/right_gripper_macro.xacro (robot description, xacro)
@@ -28,9 +28,9 @@
 		<xacro:include filename="$(find robotiq_2f_85_gripper_visualization)/urdf/robotiq_arg2f_85_model_macro.xacro" />
 		<!--Aluminium Adapter plate for Robotiq coupling and CSDA10F arm flange-->
-		<link name="${prefix}link_gripper_adapter_plate">
+		<link name="${prefix}gripper_adapter_plate">
 			<visual>
 				<origin rpy="0 0 0" xyz="0 0 0"/>
 				<geometry>
-					<mesh filename="package://invite_motoman_support/meshes/robotiq-yaskawa_adapter_plate.stl" scale="0.001 0.001 0.001"/>
+					<mesh filename="package://invite_motoman_support/meshes/visual/robotiq-yaskawa_adapter_plate.stl" scale="0.001 0.001 0.001"/>
 				</geometry>
 				<material name="Aluminium">
@@ -47,9 +47,9 @@
 		</link>
 		<!--Robotiq coupling, that connects the gripper with the Adapter plate; this part host the cable connections of the gripper-->
-		<link name="${prefix}link_robotiq_coupling">
+		<link name="${prefix}robotiq_coupling">
 			<visual>
 				<origin rpy="0 0 0" xyz="0 0 0"/>
 				<geometry>
-					<mesh filename="package://invite_motoman_support/meshes/robotiq_gripper_coupling.stl" scale="0.001 0.001 0.001"/>
+					<mesh filename="package://invite_motoman_support/meshes/visual/robotiq_gripper_coupling.stl" scale="0.001 0.001 0.001"/>
 				</geometry>
 				<material name="light_balck">
@@ -71,11 +71,11 @@
 		<joint name="${prefix}gripper_coupling_joint" type="fixed">
 			<origin  xyz="0 0.0160 0" rpy="${-pi/2} 0 0"/>
-			<parent link="${prefix}link_gripper_adapter_plate" />
-			<child link="${prefix}link_robotiq_coupling" />
+			<parent link="${prefix}gripper_adapter_plate" />
+			<child link="${prefix}robotiq_coupling" />
 		</joint>
 		<!--Joint from the robotiq coupling to the gripper itself-->
 		<joint name="${prefix}joint" type="fixed">
 			<origin xyz="0 0.0 0.0039" rpy="0 0 ${pi}" />
-			<parent link="${prefix}link_robotiq_coupling" />
+			<parent link="${prefix}robotiq_coupling" />
 			<child link="${prefix}robotiq_arg2f_base_link" />
 		</joint>

File: invite_motoman_support/urdf/urdf_macros_examples/left_gripper.xacro (robot description, xacro)
@@ -17,5 +17,5 @@
   <joint name="world_joint" type="fixed">
     <parent link="base_link" />
-    <child link="link_gripper_adapter_plate" />
+    <child link="ft300_adapter_plate" />
     <origin xyz="0 0 0" rpy="0 0 0"/>
     <axis xyz="0 0 1"/>

Commit message: v1.1.7 Minor changes, Configuration of two 85mm stroke grippers
- Change repository cover picture 
- Typos corrections 
- Organize and configure testing of grippers URDFs sepparetly
- Update self-collision matrix

File: invite_motoman_support/urdf/invite_csda10f.xacro (robot description, xacro)
@@ -47,4 +47,5 @@
 		<child link="arm_left_link_tcp" />
 	</joint>
+  <!-- TO-Do: Move to the collision scene  -->
 	<link name="ensenso_upper_optical_frame">
 		<visual>
@@ -83,6 +84,4 @@
 	<joint name="upper_camera_joint" type="fixed">
 		<origin xyz="0.860775 0.265338 1.88787" rpy="-2.89701 0.0272259 1.57315"/>
-		<!-- <origin xyz="0.865275 0.259338 1.89787" rpy="-2.89701 0.0272259 1.57315"/> -->
-		<!-- <origin xyz="0.875275 0.259338 1.89787" rpy="-2.89701 0.0272259 1.57315"/> -->
 		<parent link="base_link" />
 		<child link="ensenso_upper_optical_frame" />
@@ -90,5 +89,4 @@
 	<joint name="lower_camera_joint" type="fixed">
 		<origin xyz="0.685186 1.32848 1.41829" rpy="-1.9854 -0.00862869 -3.13558"/>
-		<!-- <origin xyz="0.695186 1.32848 1.41829" rpy="-1.9854 -0.00862869 -3.13558"/> -->
 		<parent link="base_link" />
 		<child link="ensenso_lower_optical_frame" />

File: invite_motoman_support/urdf/left_gripper_macro.xacro (robot description, xacro)
@@ -12,5 +12,5 @@
 <robot xmlns:xacro="http://ros.org/wiki/xacro">
 	<xacro:macro name="invite_csda10f_left_gripper" params="prefix">
-		<!--Import macro from 2-finger adaptative robotiq gripper-->
+		<!-- Import macro from 2-finger adaptative robotiq gripper -->
 		<xacro:include filename="$(find robotiq_2f_85_gripper_visualization)/urdf/robotiq_arg2f_85_model_macro.xacro" />
 		<!-- Import macro of Robotiq force sensor FT300 -->

File: invite_motoman_support/urdf/urdf_macros_examples/right_gripper.xacro (robot description, xacro)
@@ -16,5 +16,5 @@
   <joint name="world_joint" type="fixed">
     <parent link="base_link" />
-    <child link="arm_right_link_gripper_adapter_plate" />
+    <child link="arm_right_gripper_adapter_plate" />
     <origin xyz="0 0 0" rpy="${pi/2} 0 0"/>
     <axis xyz="0 0 1"/>
